File: _4_PCB/TAP.kicad_pcb (KiCad board)
At the start: 4 copper layers, 55.9 x 55.9 mm, 3 parts, among them J1 RJ45, J2 RJ45, J3 RJ45

Commit message: creation du PCB
Parts:
- added REF**: MountingHole_3.5mm, Mounting_Holes:MountingHole_3.5mm, F.Cu at (161.9, 76.2)
- added REF**: MountingHole_3.5mm, Mounting_Holes:MountingHole_3.5mm, F.Cu at (118.7, 76.2)
- added REF**: MountingHole_3.5mm, Mounting_Holes:MountingHole_3.5mm, F.Cu at (140.2, 119.9)
Routing:
- net Net-(J1-Pad5): track 86.8 -> 53.3 mm, vias 2 -> 0
- net Net-(J1-Pad7): track 138.9 -> 152.3 mm
- net Net-(J1-Pad3): track 96.1 -> 108.6 mm, vias 0 -> 2
- net Net-(J1-Pad1): track 103.0 -> 105.5 mm
Other:
- board text added: "VoLAB TAP-3 201703"
